Commit message: update ArUco detection and corresponding environment

File: src/mrobot_description/urdf/mrobot_rgb_camera.urdf.xacro (robot description, xacro)
@@ -6,4 +6,7 @@
             <box size="0.015 0.130 0.022"/>
           </geometry>
+          <material name="Black">
+            <color rgba="${0/255} ${0/255} ${0/255} 1.0"/>
+          </material>
         </visual>
         <collision>
@@ -30,6 +33,6 @@
           <horizontal_fov>1.3962634</horizontal_fov>
           <image>
-            <width>800</width>
-            <height>800</height>
+            <width>640</width>
+            <height>480</height>
             <format>R8G8B8</format>
           </image>
@@ -43,5 +46,5 @@
             <stddev>0.007</stddev>
           </noise>
-          <lens>
+          <!-- <lens>
             <intrinsics>
               <fx>100</fx>
@@ -51,5 +54,5 @@
               <s>0</s>
             </intrinsics>
-          </lens>
+          </lens> -->
         </camera>
         <plugin name="camera_controller" filename="libgazebo_ros_camera.so">

Commit message: add a camera frame to show the axis of marker correctly

File: src/mrobot_description/urdf/mrobot_rgb_camera.urdf.xacro (robot description, xacro)
@@ -1,73 +1,79 @@
 <robot name="mrobot" xmlns:xacro="http://wiki.ros.org/xacro">
-    <link name="camera_link">
-        <visual>
-          <origin xyz="0 0 0" rpy="0 0 0"/>
-          <geometry>
-            <box size="0.015 0.130 0.022"/>
-          </geometry>
-          <material name="Black">
-            <color rgba="${0/255} ${0/255} ${0/255} 1.0"/>
-          </material>
-        </visual>
-        <collision>
-          <origin xyz="0 0 0" rpy="0 0 0"/>
-          <geometry>
-            <box size="0.015 0.130 0.022"/>
-          </geometry>
-        </collision>
-        <inertial>
-          <origin xyz="0 0 0" rpy="0 0 0"/>
-          <mass value="0.035"/>
-          <inertia ixx="0.001"  ixy="0"  ixz="0" iyy="0.001" iyz="0" izz="0.001" />
-        </inertial>
-    </link>
-    <joint name="camera_joint" type="fixed">
-      <parent link="base_link"/>
-      <child link="camera_link"/>
-      <origin xyz="0.215 0 0.05" rpy="0 0 0"/>
-    </joint>
-    <gazebo reference="camera_link">
-      <sensor type="camera" name="camera1">
-        <update_rate>30.0</update_rate>
-        <camera name="head">
-          <horizontal_fov>1.3962634</horizontal_fov>
-          <image>
-            <width>640</width>
-            <height>480</height>
-            <format>R8G8B8</format>
-          </image>
-          <clip>
-            <near>0.02</near>
-            <far>300</far>
-          </clip>
-          <noise>
-            <type>gaussian</type>
-            <mean>0.0</mean>
-            <stddev>0.007</stddev>
-          </noise>
-          <!-- <lens>
-            <intrinsics>
-              <fx>100</fx>
-              <fy>100</fy>
-              <cx>640</cx>
-              <cy>360</cy>
-              <s>0</s>
-            </intrinsics>
-          </lens> -->
-        </camera>
-        <plugin name="camera_controller" filename="libgazebo_ros_camera.so">
-          <alwaysOn>true</alwaysOn>
-          <updateRate>0.0</updateRate>
-          <imageTopicName>image_raw</imageTopicName>
-          <cameraInfoTopicName>camera_info</cameraInfoTopicName>
-          <frameName>camera_link</frameName>
-          <hackBaseline>0.07</hackBaseline>
-          <distortionK1>0.0</distortionK1>
-          <distortionK2>0.0</distortionK2>
-          <distortionK3>0.0</distortionK3>
-          <distortionT1>0.0</distortionT1>
-          <distortionT2>0.0</distortionT2>
-        </plugin>
-      </sensor>
-    </gazebo>
+  <link name="camera_link">
+      <visual>
+        <origin xyz="0 0 0" rpy="0 0 0"/>
+        <geometry>
+          <box size="0.015 0.130 0.022"/>
+        </geometry>
+        <material name="Black">
+          <color rgba="${0/255} ${0/255} ${0/255} 1.0"/>
+        </material>
+      </visual>
+      <collision>
+        <origin xyz="0 0 0" rpy="0 0 0"/>
+        <geometry>
+          <box size="0.015 0.130 0.022"/>
+        </geometry>
+      </collision>
+      <inertial>
+        <origin xyz="0 0 0" rpy="0 0 0"/>
+        <mass value="0.035"/>
+        <inertia ixx="0.001"  ixy="0"  ixz="0" iyy="0.001" iyz="0" izz="0.001" />
+      </inertial>
+  </link>
+  <joint name="camera_joint" type="fixed">
+    <parent link="base_link"/>
+    <child link="camera_link"/>
+    <origin xyz="0.215 0 0.05" rpy="0 0 0"/>
+  </joint>
+  <link name="camera_depth_frame"/>
+  <joint name="camera_depth_joint" type="fixed">
+    <origin xyz="0 0 0" rpy="${-pi/2} 0 ${-pi/2}"/>
+    <parent link="camera_link"/>
+    <child link="camera_depth_frame"/>
+  </joint>
+  <gazebo reference="camera_link">
+    <sensor type="camera" name="camera1">
+      <update_rate>30.0</update_rate>
+      <camera name="head">
+        <horizontal_fov>1.3962634</horizontal_fov>
+        <image>
+          <width>640</width>
+          <height>480</height>
+          <format>R8G8B8</format>
+        </image>
+        <clip>
+          <near>0.02</near>
+          <far>300</far>
+        </clip>
+        <noise>
+          <type>gaussian</type>
+          <mean>0.0</mean>
+          <stddev>0.007</stddev>
+        </noise>
+        <!-- <lens>
+          <intrinsics>
+            <fx>100</fx>
+            <fy>100</fy>
+            <cx>640</cx>
+            <cy>360</cy>
+            <s>0</s>
+          </intrinsics>
+        </lens> -->
+      </camera>
+      <plugin name="camera_controller" filename="libgazebo_ros_camera.so">
+        <alwaysOn>true</alwaysOn>
+        <updateRate>0.0</updateRate>
+        <imageTopicName>image_raw</imageTopicName>
+        <cameraInfoTopicName>camera_info</cameraInfoTopicName>
+        <frameName>camera_link</frameName>
+        <hackBaseline>0.07</hackBaseline>
+        <distortionK1>0.0</distortionK1>
+        <distortionK2>0.0</distortionK2>
+        <distortionK3>0.0</distortionK3>
+        <distortionT1>0.0</distortionT1>
+        <distortionT2>0.0</distortionT2>
+      </plugin>
+    </sensor>
+  </gazebo>
 </robot>
