Commit message: update URDF model and charging station detection

File: src/mrobot_description/urdf/mrobot.urdf.xacro (robot description, xacro)
@@ -4,6 +4,6 @@
 	<xacro:include filename="mrobot_body_ros2_control.xacro"/>
 	<xacro:include filename="mrobot_body.urdf.xacro"/>
+	<xacro:include filename="mrobot_lidar.urdf.xacro"/>
 	<xacro:include filename="mrobot_imu.urdf.xacro"/>
-	<xacro:include filename="mrobot_lidar.urdf.xacro"/>
 	<xacro:include filename="mrobot_rgb_camera.urdf.xacro"/>
 </robot>

File: src/mrobot_description/urdf/mrobot_body.urdf.xacro (robot description, xacro)
@@ -1,128 +1,105 @@
 <robot name="mrobot" xmlns:xacro="http://ros.org/wiki/xacro">
-    <!-- ****************** ROBOT CONSTANTS *******************************  -->
-  <!-- Define the size of the robot's main chassis in meters -->
-  <xacro:property name="base_width" value="0.39"/>
-  <xacro:property name="base_length" value="0.70"/>
-  <xacro:property name="base_height" value="0.20"/>
-  <!-- Define the shape of the robot's two back wheels in meters -->
-  <xacro:property name="wheel_radius" value="0.14"/>
-  <xacro:property name="wheel_width" value="0.06"/>
-  <!-- x-axis points forward, y-axis points to left, z-axis points upwards -->
-  <!-- Define the gap between the wheel and chassis along y-axis in meters -->
-  <xacro:property name="wheel_ygap" value="0.035"/>
-  <!-- Position the wheels along the z-axis -->
-  <xacro:property name="wheel_zoff" value="0.05"/>
-  <!-- Position the wheels along the x-axis -->
-  <xacro:property name="wheel_xoff" value="0.221"/>
-  <!-- Position the caster wheel along the x-axis -->
-  <xacro:property name="caster_xoff" value="0.217"/>
-  <!-- Define intertial property macros  -->
-  <xacro:macro name="box_inertia" params="m w h d">
-    <inertial>
-      <origin xyz="0 0 0" rpy="${pi/2} 0 ${pi/2}"/>
-      <mass value="${m}"/>
-      <inertia ixx="${(m/12) * (h*h + d*d)}" ixy="0.0" ixz="0.0" iyy="${(m/12) * (w*w + d*d)}" iyz="0.0" izz="${(m/12) * (w*w + h*h)}"/>
-    </inertial>
-  </xacro:macro>
-  <xacro:macro name="cylinder_inertia" params="m r h">
-    <inertial>
-      <origin xyz="0 0 0" rpy="${pi/2} 0 0" />
-      <mass value="${m}"/>
-      <inertia ixx="${(m/12) * (3*r*r + h*h)}" ixy = "0" ixz = "0" iyy="${(m/12) * (3*r*r + h*h)}" iyz = "0" izz="${(m/2) * (r*r)}"/>
-    </inertial>
-  </xacro:macro>
-  <xacro:macro name="sphere_inertia" params="m r">
-    <inertial>
-      <mass value="${m}"/>
-      <inertia ixx="${(2/5) * m * (r*r)}" ixy="0.0" ixz="0.0" iyy="${(2/5) * m * (r*r)}" iyz="0.0" izz="${(2/5) * m * (r*r)}"/>
-    </inertial>
-  </xacro:macro>
-  <!-- ********************** ROBOT BASE *********************************  -->
+  <!-- base_footprint -->
+  <link name="base_footprint"/>
+  <!-- base_link -->
   <link name="base_link">
-    <visual>
-      <geometry>
-        <box size="${base_length} ${base_width} ${base_height}"/>
-      </geometry>
-      <material name="Red">
-        <color rgba="${255/255} ${0/255} ${0/255} 1.0"/>
-      </material>
-    </visual>
-    <collision>
-      <geometry>
-        <box size="${base_length} ${base_width} ${base_height}"/>
-      </geometry>
-    </collision>
-    <xacro:box_inertia m="10.0" w="${base_width}" d="${base_length}" h="${base_height}"/>
-  </link>
-  <!-- ****************** ROBOT BASE FOOTPRINT ***************************  -->
-  <!-- Define the center of the main robot chassis projected on the ground -->
-  <link name="base_footprint">
-  </link>
-  <!-- The base footprint of the robot is located underneath the chassis -->
-  <joint name="base_joint" type="fixed">
-    <parent link="base_footprint"/>
-    <child link="base_link" />
-    <origin xyz="0.0 0.0 ${(wheel_radius+wheel_zoff)}" rpy="0 0 0"/>
-  </joint>
-  <!-- *********************** DRIVE WHEELS ******************************  -->
-  <xacro:macro name="wheel" params="prefix x_reflect y_reflect">
-    <link name="${prefix}_link">
+      <inertial>
+          <origin xyz="-1.51807472482668E-05 2.79346181472073E-05 0.0866200775222906" rpy="0 0 0" />
+          <mass value="64.7171962068877" />
+          <inertia ixx="1.42225890496994" ixy="-0.000392754943773645" ixz="0.0708650035684445"
+                   iyy="3.51249641237205" iyz="-0.000160647777377098" izz="4.57970566976989" />
+      </inertial>
       <visual>
-        <origin xyz="0 0 0" rpy="${pi/2} 0 0"/>
-        <geometry>
-            <cylinder radius="${wheel_radius}" length="${wheel_width}"/>
-        </geometry>
-        <material name="White">
-          <color rgba="${255/255} ${255/255} ${255/255} 1.0"/>
-        </material>
+          <origin xyz="0 0 0" rpy="0 0 0" />
+          <geometry>
+            <mesh filename="package://mrobot_description/meshes/base_link.STL" />
+          </geometry>
+          <material name="">
+            <color rgba="0.792156862745098 0.819607843137255 0.933333333333333 1" />
+          </material>
       </visual>
       <collision>
-        <origin xyz="0 0 0" rpy="${pi/2} 0 0"/>
-        <geometry>
-          <cylinder radius="${wheel_radius}" length="${wheel_width}"/>
-        </geometry>
+          <origin xyz="0 0 0" rpy="0 0 0" />
+          <geometry>
+            <mesh filename="package://mrobot_description/meshes/base_link.STL" />
+          </geometry>
       </collision>
-      <xacro:cylinder_inertia m="0.5" r="${wheel_radius}" h="${wheel_width}"/>
+  </link>
+  <!-- base_footprint -> base_link joint -->
+  <joint name="base_footprint_joint" type="fixed">
+      <origin xyz="0 0 0" rpy="0 0 0"/>
+      <parent link="base_footprint"/>
+      <child link="base_link"/>
+  </joint>
+  <!-- Wheel and joint macro -->
+  <xacro:macro name="wheel" params="name inertial_xyz joint_xyz">
+      <link name="${name}_wheel">
+        <inertial>
+            <origin xyz="${inertial_xyz}" rpy="0 0 0" />
+            <mass value="0.99202" />
+            <inertia ixx="0.0017289" ixy="-1.1999E-19" ixz="2.0419E-19"
+                      iyy="0.0030122" iyz="4.5246E-18" izz="0.0017289" />
+        </inertial>
+        <visual>
+            <origin xyz="0 0 0" rpy="0 0 0" />
+            <geometry>
+                <mesh filename="package://mrobot_description/meshes/${name}_wheel.STL" />
+            </geometry>
+            <material name="">
+                <color rgba="0.79216 0.81961 0.93333 1" />
+            </material>
+        </visual>
+        <collision>
+            <origin xyz="0 0 0" rpy="0 0 0" />
+            <geometry>
+                <mesh filename="package://mrobot_description/meshes/${name}_wheel.STL" />
+            </geometry>
+        </collision>
+      </link>
+      <joint name="${name}_wheel_joint" type="continuous">
+        <origin xyz="${joint_xyz}" rpy="0 0 0" />
+        <parent link="base_link" />
+        <child link="${name}_wheel" />
+        <axis xyz="0 1 0" />
+      </joint>
+    </xacro:macro>
+  <!-- Create left and right wheel/joint -->
+  <xacro:wheel name="right" inertial_xyz="-1.1102E-16 0.026 2.2204E-16" joint_xyz="-0.1621 -0.242 0.066"  />
+  <xacro:wheel name="left" inertial_xyz="-1.1102E-16 -0.026 -1.6653E-16" joint_xyz="-0.1621 0.242 0.066" />
+  <!-- Caster wheel and joint macro -->
+  <xacro:macro name="caster" params="name inertial_xyz joint_xyz">
+    <link name="${name}_caster">
+      <inertial>
+          <origin xyz="${inertial_xyz}" rpy="0 0 0" />
+          <mass value="0.25623" />
+          <inertia ixx="0.00017108" ixy="-2.4081E-10" ixz="-5.2581E-12"
+                    iyy="0.00016998" iyz="1.9178E-19" izz="0.00027267" />
+      </inertial>
+      <visual>
+          <origin xyz="0 0 0" rpy="0 0 0" />
+          <geometry>
+              <mesh filename="package://mrobot_description/meshes/${name}_caster.STL" />
+          </geometry>
+          <material name="">
+              <color rgba="0.79216 0.81961 0.93333 1" />
+          </material>
+      </visual>
+      <collision>
+          <origin xyz="0 0 0" rpy="0 0 0" />
+          <geometry>
+              <mesh filename="package://mrobot_description/meshes/${name}_caster.STL" />
+          </geometry>
+      </collision>
     </link>
-    <!-- Connect the wheels to the base_link at the appropriate location, and
-         define a continuous joint to allow the wheels to freely rotate about
-         an axis -->
-    <joint name="${prefix}_joint" type="continuous">
-      <parent link="base_link"/>
-      <child link="${prefix}_link"/>
-      <origin xyz="${x_reflect*wheel_xoff} ${y_reflect*(base_width/2+wheel_ygap)} ${-wheel_zoff}" rpy="0 0 0"/>
-      <axis xyz="0 1 0"/>
+    <joint name="base_to_${name}_caster" type="continuous">
+      <origin xyz="${joint_xyz}" rpy="0 0 0" />
+      <parent link="base_link" />
+      <child link="${name}_caster" />
+      <axis xyz="0 0 1" />
     </joint>
   </xacro:macro>
-  <!-- Instantiate two wheels using the macro we just made through the
-       xacro:wheel tags. We also define the parameters to have one wheel
-       on both sides at the back of our robot (i.e. x_reflect=-1). -->
-  <xacro:wheel prefix="drivewhl_l" x_reflect="-1" y_reflect="1" />
-  <xacro:wheel prefix="drivewhl_r" x_reflect="-1" y_reflect="-1" />
-  <!-- *********************** CASTER WHEEL ******************************  -->
-  <!-- We add a caster wheel. It will be modeled as sphere.
-       We define the wheel’s geometry, material and the joint to connect it to
-       base_link at the appropriate location. -->
-  <link name="front_caster">
-    <visual>
-      <geometry>
-        <sphere radius="${(wheel_radius+wheel_zoff-(base_height/2))}"/>
-      </geometry>
-      <material name="White">
-        <color rgba="${255/255} ${255/255} ${255/255} 1.0"/>
-      </material>
-    </visual>
-    <collision>
-      <origin xyz="0 0 0" rpy="0 0 0"/>
-      <geometry>
-        <sphere radius="${(wheel_radius+wheel_zoff-(base_height/2))}"/>
-      </geometry>
-    </collision>
-    <xacro:sphere_inertia m="0.05" r="${(wheel_radius+wheel_zoff-(base_height/2))}"/>
-  </link>
-  <joint name="caster_joint" type="fixed">
-    <parent link="base_link"/>
-    <child link="front_caster"/>
-    <origin xyz="${caster_xoff} 0.0 ${-(base_height/2)}" rpy="0 0 0"/>
-  </joint>
+  <!-- Create 3 caster wheels -->
+  <xacro:caster name="left" inertial_xyz="8.9465E-08 -5.5511E-17 0.019764" joint_xyz="0.3504 0.18406 0"/>
+  <xacro:caster name="right" inertial_xyz="8.9465E-08 -2.2204E-16 0.019764" joint_xyz="0.35023 -0.18491 0"/>
+  <xacro:caster name="back" inertial_xyz="8.9465E-08 0 0.019764" joint_xyz="-0.31668 -0.0019708 0"/>
 </robot>

File: src/mrobot_description/urdf/mrobot_body_gazebo.xacro (robot description, xacro)
@@ -1,48 +1,66 @@
 <?xml version="1.0"?>
 <robot name="mrobot" xmlns:xacro="http://ros.org/wiki/xacro">
-    <transmission name="drivewhl_l_transmission">
+    <transmission name="left_wheel_transmission">
         <type>transmission_interface/SimpleTransmission</type>
-        <actuator name="drivewhl_l_motor" role="actuator_drivewhl_l"/>
-        <joint name="drivewhl_l_joint" role="joint_drivewhl_l">
+        <actuator name="left_wheel_motor" role="left_wheel_actuator"/>
+        <joint name="left_wheel_joint" role="joint_left">
             <mechanical_reduction>1.0</mechanical_reduction>
         </joint>
     </transmission>
-    <transmission name="drivewhl_r_transmission">
+    <transmission name="right_wheel_transmission">
         <type>transmission_interface/SimpleTransmission</type>
-        <actuator name="drivewhl_r_motor" role="actuator_drivewhl_r"/>
-        <joint name="drivewhl_r_joint" role="joint_drivewhl_r">
+        <actuator name="right_wheel_motor" role="right_wheel_actuator"/>
+        <joint name="right_wheel_joint" role="joint_right">
             <mechanical_reduction>1.0</mechanical_reduction>
         </joint>
     </transmission>
-    <gazebo reference="drivewhl_l_link">
-        <mu1>100000000000000.0</mu1>
-        <mu2>100000000000000.0</mu2>
+    <gazebo reference="left_wheel">
+        <mu1>1000000000000000.0</mu1>
+        <mu2>1000000000000000.0</mu2>
         <kp>1000000000000.0</kp>
-        <kd>10.0</kd>
+        <kd>100.0</kd>
+        <maxVel>0.1</maxVel>
+        <fdir1>1 0 0</fdir1>
+        <material>Gazebo/Black</material>
+    </gazebo>
+    <gazebo reference="right_wheel">
+        <mu1>1000000000000000.0</mu1>
+        <mu2>1000000000000000.0</mu2>
+        <kp>1000000000000.0</kp>
+        <kd>100.0</kd>
         <minDepth>0.001</minDepth>
         <maxVel>0.1</maxVel>
         <fdir1>1 0 0</fdir1>
-        <material>Gazebo/White</material>
+        <material>Gazebo/Black</material>
     </gazebo>
-    <gazebo reference="drivewhl_r_link">
-        <mu1>100000000000000.0</mu1>
-        <mu2>100000000000000.0</mu2>
-        <kp>1000000000000.0</kp>
-        <kd>10.0</kd>
-        <minDepth>0.001</minDepth>
-        <maxVel>0.1</maxVel>
-        <fdir1>1 0 0</fdir1>
-        <material>Gazebo/White</material>
-    </gazebo>
-    <gazebo reference="front_caster">
+    <gazebo reference="left_caster">
         <mu1>0.1</mu1>
         <mu2>0.1</mu2>
         <kp>1000000.0</kp>
         <kd>100.0</kd>
+        <minDepth>0.001</minDepth>
+        <maxVel>1.0</maxVel>
+        <material>Gazebo/White</material>
+    </gazebo>
+    <gazebo reference="right_caster">
+        <mu1>0.1</mu1>
+        <mu2>0.1</mu2>
+        <kp>1000000.0</kp>
+        <kd>100.0</kd>
+        <minDepth>0.001</minDepth>
+        <maxVel>1.0</maxVel>
+        <material>Gazebo/White</material>
+    </gazebo>
+    <gazebo reference="back_caster">
+        <mu1>0.1</mu1>
+        <mu2>0.1</mu2>
+        <kp>1000000.0</kp>
+        <kd>100.0</kd>
+        <minDepth>0.001</minDepth>
         <maxVel>1.0</maxVel>
         <material>Gazebo/White</material>
     </gazebo>
     <gazebo reference="base_link">
-        <material>Gazebo/Red</material>
+        <material>Gazebo/Yellow</material>
     </gazebo>
     <gazebo>

File: src/mrobot_description/urdf/mrobot_body_ros2_control.xacro (robot description, xacro)
@@ -5,5 +5,5 @@
             <plugin>gazebo_ros2_control/GazeboSystem</plugin>
         </hardware>
-        <joint name="drivewhl_l_joint">
+        <joint name="left_wheel_joint">
             <command_interface name="velocity">
                 <param name="min">-1</param>
@@ -13,5 +13,5 @@
             <state_interface name="velocity"/>
         </joint>
-        <joint name="drivewhl_r_joint">
+        <joint name="right_wheel_joint">
             <command_interface name="velocity">
                 <param name="min">-1</param>

File: src/mrobot_description/urdf/mrobot_imu.urdf.xacro (robot description, xacro)
@@ -1,21 +1,29 @@
 <robot name="mrobot" xmlns:xacro="http://wiki.ros.org/xacro">
+    <!-- Define intertial property macros  -->
+    <xacro:macro name="box_inertia" params="m w h d">
+        <inertial>
+        <origin xyz="0 0 0" rpy="${pi/2} 0 ${pi/2}"/>
+        <mass value="${m}"/>
+        <inertia ixx="${(m/12) * (h*h + d*d)}" ixy="0.0" ixz="0.0" iyy="${(m/12) * (w*w + d*d)}" iyz="0.0" izz="${(m/12) * (w*w + h*h)}"/>
+        </inertial>
+    </xacro:macro>
     <!-- imu -->
     <link name="imu_link">
         <visual>
         <geometry>
-            <box size="0.1 0.1 0.1"/>
+            <box size="0.05 0.05 0.05"/>
         </geometry>
         </visual>
         <collision>
         <geometry>
-            <box size="0.1 0.1 0.1"/>
+            <box size="0.05 0.05 0.05"/>
         </geometry>
         </collision>
-        <xacro:box_inertia m="0.1" w="0.1" d="0.1" h="0.1"/>
+        <xacro:box_inertia m="0.01" w="0.05" d="0.05" h="0.05"/>
     </link>
     <joint name="imu_joint" type="fixed">
         <parent link="base_link"/>
         <child link="imu_link"/>
-        <origin xyz="0 0 0.01"/>
+        <origin xyz="0 0 0.10"/>
     </joint>
     <gazebo reference="imu_link">

File: src/mrobot_description/urdf/mrobot_lidar.urdf.xacro (robot description, xacro)
@@ -1,61 +1,70 @@
 <!-- lidar-->
 <robot name="mrobot" xmlns:xacro="http://wiki.ros.org/xacro">
-    <link name="lidar_link">
-        <inertial>
-          <origin xyz="0 0 0" rpy="0 0 0"/>
-          <mass value="0.125"/>
-          <inertia ixx="0.001"  ixy="0"  ixz="0" iyy="0.001" iyz="0" izz="0.001" />
-        </inertial>
-        <collision>
-          <origin xyz="0 0 0" rpy="0 0 0"/>
-          <geometry>
-             <cylinder radius="0.0508" length="0.055"/>
-          </geometry>
-        </collision>
-        <visual>
-          <origin xyz="0 0 0" rpy="0 0 0"/>
-          <geometry>
-             <cylinder radius="0.0508" length="0.055"/>
-          </geometry>
-        </visual>
+  <xacro:macro name="lidar" params="name inertial_xyz joint_xyz joint_rpy">
+      <link name="${name}_lidar">
+          <inertial>
+              <origin xyz="${inertial_xyz}" rpy="0 0 0" />
+              <mass value="0.31659" />
+              <inertia ixx="0.00022501" ixy="-7.9146E-11" ixz="-7.5617E-11"
+                        iyy="0.000225" iyz="-5.4184E-19" izz="0.00031918" />
+          </inertial>
+          <visual>
+              <origin xyz="0 0 0" rpy="0 0 0" />
+              <geometry>
+                  <mesh filename="package://mrobot_description/meshes/${name}_lidar.STL" />
+              </geometry>
+              <material name="">
+                  <color rgba="0.79216 0.81961 0.93333 1" />
+              </material>
+          </visual>
+          <collision>
+              <origin xyz="0 0 0" rpy="0 0 0" />
+              <geometry>
+                  <mesh filename="package://mrobot_description/meshes/${name}_lidar.STL" />
+              </geometry>
+          </collision>
       </link>
-      <joint name="lidar_joint" type="fixed">
-        <parent link="base_link"/>
-        <child link="lidar_link"/>
-        <origin xyz="0 0 0.12" rpy="0 0 0"/>
+      <joint name="base_to_${name}_lidar" type="fixed">
+          <origin xyz="${joint_xyz}" rpy="${joint_rpy}" />
+          <parent link="base_link" />
+          <child link="${name}_lidar" />
+          <axis xyz="0 0 0" />
       </joint>
-      <gazebo reference="lidar_link">
-        <sensor name="lidar" type="ray">
-          <always_on>true</always_on>
-          <visualize>true</visualize>
-          <update_rate>5</update_rate>
-          <ray>
-            <scan>
-              <horizontal>
-                <samples>360</samples>
-                <resolution>1.000000</resolution>
-                <min_angle>0.000000</min_angle>
-                <max_angle>6.280000</max_angle>
-              </horizontal>
-            </scan>
-            <range>
-              <min>0.120000</min>
-              <max>3.5</max>
-              <resolution>0.015000</resolution>
-            </range>
-            <noise>
-              <type>gaussian</type>
-              <mean>0.0</mean>
-              <stddev>0.01</stddev>
-            </noise>
-          </ray>
-          <plugin name="scan" filename="libgazebo_ros_ray_sensor.so">
-            <ros>
-              <remapping>~/out:=scan</remapping>
-            </ros>
-            <output_type>sensor_msgs/LaserScan</output_type>
-            <frame_name>lidar_link</frame_name>
-          </plugin>
-        </sensor>
-      </gazebo>
+  </xacro:macro>
+  <!-- create lidar -->
+  <xacro:lidar name="front" inertial_xyz="9.7076E-09 0 0.024888" joint_xyz="0.2379 0 0.1802" joint_rpy="0 0 0"/>
+  <gazebo reference="front_lidar">
+    <sensor name="lidar" type="ray">
+      <always_on>true</always_on>
+      <visualize>true</visualize>
+      <update_rate>5</update_rate>
+      <ray>
+        <scan>
+          <horizontal>
+            <samples>360</samples>
+            <resolution>1.000000</resolution>
+            <min_angle>-1.570796</min_angle>
+            <max_angle>1.570796</max_angle>
+          </horizontal>
+        </scan>
+        <range>
+          <min>0.120000</min>
+          <max>3.5</max>
+          <resolution>0.015000</resolution>
+        </range>
+        <noise>
+          <type>gaussian</type>
+          <mean>0.0</mean>
+          <stddev>0.01</stddev>
+        </noise>
+      </ray>
+      <plugin name="scan" filename="libgazebo_ros_ray_sensor.so">
+        <ros>
+          <remapping>~/out:=scan</remapping>
+        </ros>
+        <output_type>sensor_msgs/LaserScan</output_type>
+        <frame_name>front_lidar</frame_name>
+      </plugin>
+    </sensor>
+  </gazebo>
 </robot>

File: src/mrobot_description/urdf/mrobot_rgb_camera.urdf.xacro (robot description, xacro)
@@ -25,5 +25,5 @@
     <parent link="base_link"/>
     <child link="camera_link"/>
-    <origin xyz="0.215 0 0.05" rpy="0 0 0"/>
+    <origin xyz="0.31 0 0.15" rpy="0 0 0"/>
   </joint>
   <link name="camera_depth_frame"/>
@@ -39,6 +39,6 @@
         <horizontal_fov>1.3962634</horizontal_fov>
         <image>
-          <width>640</width>
-          <height>480</height>
+          <width>800</width>
+          <height>800</height>
           <format>R8G8B8</format>
         </image>
